File: KiCAD-PCB/Version20260523/ESP32C6_gasometer-2026-07-11_162129/ESP32C6_gasometer.kicad_sch (KiCad schematic)
At the start: 14 parts, among them J1 JST-SH 1.25 2pin plug, J2 JST-SH 1.25 2pin socket, SW1 KSK-1A87-2025, SW2 OMRON_B3F-6000, SW3 OMRON_B3F-6000, U1 TPL5110, U2 XIAO-ESP32-C6

Commit message: docs(kicad): Reed-Empfindlichkeit und Steckerpraezisierung
- Praezisierung der Reed-Schalter Empfindlichkeit *-1520, anstatt *-2025
- Akku-Buchse JST-PH2.0
- Reed-Schalter Stecker/Buchse JST-XH1.25

Co-authored-by: Cursor <cursoragent@cursor.com>
Parts:
- SW1: value KSK-1A87-2025 -> KSK-1A87-1520
Changed lines of the file:
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@@
 			)
 		)
-		(property "Value" "KSK-1A87-2025"
+		(property "Value" "KSK-1A87-1520"
 			(at 26.67 76.1999 90)
 			(show_name no)
